File: rocket_nose_selfie_camera.kicad_sch (KiCad schematic)
At the start: 15 parts, among them J1 LOGGER TRIGGER / STATUS, J3 LOGGER CAN, J4 POWER IN: +5V/GND (power boar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, U2 MCP2562-E/SN, U3 XIAO-ESP32-S3-SMD

Commit message: sch: power CAN transceiver from XIAO 3V3 (SN65HVD230)
- Replace U2 MCP2562-E/SN with SN65HVD230DR, VCC from +3.3V (C1 100 nF), Rs to GND, Vref NC
- Remove C2; 5V_IN now feeds only D3, so CAN works on USB power alone without J4
- Add mounting holes H1-H4 and board setup defaults
- Sync README and BOM

Note: deviates from the global CAN transceiver preference (MCP2562-E-SN);
SN65HVD230 is not stocked at Akizuki/Sengoku. PCB not yet updated from schematic.
Parts:
- removed C2: 100nF, Capacitor_SMD:C_0603_1608Metric, symbol Device:C
- removed U2: MCP2562-E/SN, Package_SO:SOIC-8_3.9x4.9mm_P1.27mm, symbol Interface_CAN_LIN:MCP2562-E-SN
- added H1, H2, H3, H4: M2, MountingHole:MountingHole_2.2mm_M2, symbol Mechanical:MountingHole
- added U2: SN65HVD230DR, Package_SO:SOIC-8_3.9x4.9mm_P1.27mm, symbol Interface_CAN_LIN:SN65HVD230
- D1, R3: kicad_auto_layout_block_id power_indicator -> block.u3
- D2, R4: kicad_auto_layout_block_id status_output -> block.u3
- D3: kicad_auto_layout_block_id status_output -> camera_harness
- U3: kicad_auto_layout_block_id (none) -> block.u3
Connections:
- net +3.3V: now also C1.2, U2.3 (VCC)
- net 5V_IN: no longer C1.2
- net CANH: now also U2.7 (CANH)
- net CANL: now also U2.6 (CANL)
- net CAN_RX: now also U2.4 (R)
- net CAN_TX: now also U2.1 (D)
- net GND: now also U2.2 (GND), U2.8 (Rs)
- no-connect marks 15 -> 16
Other:
- note added: "BLOCK 3 — LOGGER CAN (SN65HVD230, 3.3V)"
- note added: "Power: J4 5V_IN -> D3 (B5819W) -> XIAO VBUS; U2 runs from XIAO +3.3V."
- note removed: "BLOCK 3 — LOGGER CAN (MCP2562-E/SN)"
- note removed: "Power: J4 5V_IN -> D3 (B5819W) -> XIAO VBUS; 5V_IN also feeds U2 VDD directly."
